Commit message: +submit working simulation

File: description/robot_core.xacro (robot description, xacro)
@@ -40,4 +40,7 @@
     </xacro:inertial_box>
     </link>
+    <gazebo reference="chassis">
+        <material>Gazebo/Orange</material>
+    </gazebo>
     <!-- LEFT WHEEL LINK - 0.175 the value move to Y from 0 for our wheel, Z is rotation of the wheel-->
     <joint name="left_wheel_joint" type="continuous">
@@ -63,4 +66,7 @@
     </xacro:inertial_cylinder>
     </link>
+    <gazebo reference="left_wheel">
+        <material>Gazebo/Blue</material>
+    </gazebo>
     <!-- RIGHT WHEEL LINK - 0.175 the value move to Y from 0 for our wheel, Z is rotation of the wheel-->
     <joint name="right_wheel_joint" type="continuous">
@@ -86,4 +92,7 @@
     </xacro:inertial_cylinder>
     </link>
+    <gazebo reference="right_wheel">
+        <material>Gazebo/Blue</material>
+    </gazebo>
     <!-- CASTER WHEEL LINK -->
     <joint name="caster_wheel_joint" type="fixed">
@@ -108,3 +117,8 @@
     </xacro:inertial_sphere>
     </link>
+    <gazebo reference="caster_wheel">
+        <material>Gazebo/Black</material>
+        <mu1 value="0.001"/>
+        <mu2 value="0.001"/>
+    </gazebo>
 </robot>
